File: Hardware/LoraMulty/rns-gate.kicad_pcb (KiCad board)
At the start: 2 copper layers, 48 x 46 mm, 19 parts, among them J2 Conn_02x13_Odd_Even, U1 E22-900M30S-SX1262, U2 TCA9554PW

Commit message: refactor: fix typo in file
Other:
- board text added: "RNS-Gate de R1CBU Lora Multi module"
- board text removed: "RNS-Gate de R1CBU Lora Multy module"
Changed lines of the file:
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@@
   (gr_arc (start 206.8 50.81) (mid 208.992031 51.717969) (end 209.9 53.91) (layer "Edge.Cuts") (width 0.05))
   (gr_line (start 209.9 92.352) (end 209.9 93.71) (layer "Edge.Cuts") (width 0.05))
-  (gr_text "RNS-Gate de R1CBU\nLora Multy module" (at 194.79 55.7784) (layer "F.SilkS")
+  (gr_text "RNS-Gate de R1CBU\nLora Multi module" (at 194.79 55.7784) (layer "F.SilkS")
     (effects (font (size 1 1) (thickness 0.15)))
   )
