File: Hardware/Audio/rns-gate.kicad_sch (KiCad schematic)
At the start: 17 parts, among them J1 Conn_01x13, J2 Conn_02x13_Odd_Even, J3 Conn_01x02, J5 Conn_01x04, Q1 2N7002

Commit message: Clarification in the Audio module schematic
Parts:
- R3: value tune -> 4k3
- R4: value tune -> 680
- R5, R6: value tune -> 2k4
Other:
- note added: "Install RV1 or R3+R4"
- note added: "Install RV2 or R5+R6"
Changed lines of the file:
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@@
     (stroke (width 0) (type default) (color 0 0 0 0))
+  )
+  (text "Install RV1 or R3+R4\n" (at 112.268 101.854 0)
+    (effects (font (size 1.27 1.27)) (justify left bottom))
+  )
+  (text "Install RV2 or R5+R6\n" (at 103.378 67.564 0)
+    (effects (font (size 1.27 1.27)) (justify left bottom))
   )
   (symbol (lib_id "Device:C_Small") (at 91.44 72.39 90) (unit 1)
@@
       (effects (font (size 1.27 1.27)) (justify right))
     )
-    (property "Value" "tune" (id 1) (at 92.202 107.696 0)
+    (property "Value" "680" (id 1) (at 92.202 107.696 0)
       (effects (font (size 1.27 1.27)) (justify right))
     )
@@
       (effects (font (size 1.27 1.27)) (justify right))
     )
-    (property "Value" "tune" (id 1) (at 92.202 97.282 0)
+    (property "Value" "4k3" (id 1) (at 92.202 97.282 0)
       (effects (font (size 1.27 1.27)) (justify right))
     )
@@
       (effects (font (size 1.27 1.27)) (justify right))
     )
-    (property "Value" "tune" (id 1) (at 111.76 77.7239 0)
+    (property "Value" "2k4" (id 1) (at 111.76 77.7239 0)
       (effects (font (size 1.27 1.27)) (justify right))
     )
@@
       (effects (font (size 1.27 1.27)) (justify right))
     )
-    (property "Value" "tune" (id 1) (at 111.76 86.1059 0)
+    (property "Value" "2k4" (id 1) (at 111.76 86.1059 0)
       (effects (font (size 1.27 1.27)) (justify right))
     )
@@
     )
     (path "/87cf124b-d05b-40f9-be97-8a54d3814aff"
-      (reference "R3") (unit 1) (value "tune") (footprint "Resistor_SMD:R_0805_2012Metric")
+      (reference "R3") (unit 1) (value "4k3") (footprint "Resistor_SMD:R_0805_2012Metric")
     )
     (path "/078c5c59-2171-44ad-b103-0936b04cf347"
-      (reference "R4") (unit 1) (value "tune") (footprint "Resistor_SMD:R_0805_2012Metric")
+      (reference "R4") (unit 1) (value "680") (footprint "Resistor_SMD:R_0805_2012Metric")
     )
     (path "/939b0597-1658-4175-b220-5314baf8a978"
-      (reference "R5") (unit 1) (value "tune") (footprint "Resistor_SMD:R_0805_2012Metric")
+      (reference "R5") (unit 1) (value "2k4") (footprint "Resistor_SMD:R_0805_2012Metric")
     )
     (path "/dd0e1d9b-ac55-4045-9a49-09b8cd1bbcee"
-      (reference "R6") (unit 1) (value "tune") (footprint "Resistor_SMD:R_0805_2012Metric")
+      (reference "R6") (unit 1) (value "2k4") (footprint "Resistor_SMD:R_0805_2012Metric")
     )
     (path "/a5d7b8a1-53cd-4200-b07c-c4505ef74bc7"
